Commit message: Adding Perception Files

File: gp_sim2/urdf/SimplifiedAssembly_control.urdf (robot description, URDF)
Before this commit: robot SimplifiedAssembly, 13 links, 12 joints
Links:
- added link base_link, mass 0; collision box size=0.001 0.001 0.001; visual box size=0.001 0.001 0.001
- added link camera_link, mass 1e-5; collision box size=0.073000 0.276000 0.072000; visual mesh filename=package://gp_description2/meshes/kinect.dae
Joints:
- added joint add_joint: type fixed, parent base_link, child a, origin xyz=-0.19 -0.28 0.14325 rpy=0 0 0, axis 0 0 1
- added joint camera_joint: type fixed, parent a, child camera_link, origin xyz=0.19 0 -0.02 rpy=0 0 -1.57, axis 0 0 1

Commit message: Added new urdf and fixed few frames

File: gp_sim2/urdf/SimplifiedAssembly_control.urdf (robot description, URDF)
Before this commit: robot SimplifiedAssembly, 15 links, 14 joints
Links:
- removed link base_link
- added link camera_depth_frame, mass 0.001
- added link camera_depth_optical_frame, mass 0.001
- added link camera_rgb_frame, mass 0.001
- added link camera_rgb_optical_frame, mass 0.001
- link camera_link: mass 1e-5 -> 0.001; geometry collision box size=0.07271 0.27794 0.073; visual mesh filename=package://gp_description2/meshes/kinect.dae
Joints:
- removed joint add_joint
- added joint camera_depth_joint: type fixed, parent camera_rgb_frame, child camera_depth_frame, origin xyz=0 0.0 0 rpy=0 0 0
- added joint camera_depth_optical_joint: type fixed, parent camera_depth_frame, child camera_depth_optical_frame, origin xyz=0 0 0 rpy=-1.57079632679 0 -1.57079632679
- added joint camera_rgb_joint: type fixed, parent a, child camera_rgb_frame, origin xyz=0.19 0 -0.02 rpy=0 0 3.14
- added joint camera_rgb_optical_joint: type fixed, parent camera_rgb_frame, child camera_rgb_optical_frame, origin xyz=0 0 0 rpy=-1.57079632679 0 -1.57079632679
- joint camera_joint: axis 0 0 1 -> (none); origin xyz=0.19 0 -0.02 rpy=0 0 -1.57 -> xyz=-0.031 -0.0 -0.016 rpy=0 0 0; parent a -> camera_rgb_frame

Commit message: added a few preception data

File: gp_sim2/urdf/SimplifiedAssembly_control.urdf (robot description, URDF)
Before this commit: robot SimplifiedAssembly, 18 links, 17 joints
Joints:
- joint camera_depth_joint: origin xyz=0 0.0 0 rpy=0 0 0 -> xyz=0 0.0 0 rpy=0 0 1.57
